File: moire.brd (EAGLE design)
At the start: 39.4 x 106.7 mm, 121 parts, among them IC2 LD2981ABU33, IC3 4051PW, IC5 LM4040B10, IC6 R-78E3.3-0.5, J1 PJ301_THONKICONN6, J10 PJ301_THONKICONN6, J11 PJ301_THONKICONN6, J12 PJ301_THONKICONN6, J2 PJ301_THONKICONN6, J3 PJ301_THONKICONN6, J4 PJ301_THONKICONN6, J5 PJ301_THONKICONN6, J6 PJ301_THONKICONN6, J7 PJ301_THONKICONN6, J8 PJ301_THONKICONN6, J9 PJ301_THONKICONN6, Q2 8MHz, U1 STM32F303K8T6, U2 MCP6004_SMD, U3 MCP6002_, U4 TL074_SMD, U5 TL072_SMD

Commit message: update sch
Parts:
- added C10, C17, C23, C24, C30, C33, C50, C8, C9: 100n, rcl:C0402
- added C11, C7: 22u, rcl:C1206
- added IC1: TLC59281DBQ, og-ics:TSSOP24_0635
- added L2: (no value), wuerth-elektronik:0603
- added LED10, LED11, LED12: SSL-LX3059IGW-CA, og-leds:LED-BICOLOR-THROUGHHOLE-LUMEX
- added R50: 10k, rcl:R0402
- moved LED9 373.2 mm to (-70.6, -260.1)
- moved LED7 373.0 mm to (-83.3, -260.1)
- moved LED8 368.2 mm to (-77.0, -260.1)
Connections:
- removed net +3V1: C37.1, C39.1, C40.1, C42.1, U1.1, U1.17
- removed net A_LED_1: R19.2
- removed net B_LED_1: R30.2
- removed net C_LED_1: R31.2
- removed net GRN: LED7.GREEN_C, LED8.GREEN_C, LED9.GREEN_C
- removed net LID1: Q2.2
- removed net LID2: Q2.4
- removed net N$102: R29.B, R31.1
- removed net N$103: R28.B, R30.1
- removed net RED: LED7.RED_C, LED8.RED_C, LED9.RED_C
- removed net SW_MODE_1: SW1.3, SW1.4
- removed net SW_MODE_2: SW2.3, SW2.4
- removed net SW_MODE_3: SW3.3, SW3.4
- removed net V+: U2.4, U3.8, U4.4, U5.8
- removed net V-: U2.11, U3.4, U4.11, U5.4
- new net LEDS_SCK: IC1.3, U1.26
- new net LEDS_SIN: IC1.2, U1.28
- new net N$101: IC1.9, LED7.GREEN_C
- new net N$32: IC1.11, LED8.GREEN_C
- new net N$33: IC1.10, LED7.RED_C
- new net N$34: IC1.12, LED8.RED_C
- new net N$35: IC1.7, LED9.RED_C
- new net N$36: IC1.8, LED9.GREEN_C
- new net N$37: IC1.15, LED11.RED_C
- new net N$38: IC1.16, LED11.GREEN_C
- new net N$39: IC1.13, LED10.GREEN_C
- new net N$40: IC1.17, LED12.RED_C
- new net N$42: IC1.18, LED12.GREEN_C
- new net N$43: IC1.14, LED10.RED_C
- new net N$44: C7.1, C8.1, IC1.24, L2.1
- new net N$45: IC1.19, R19.2
- new net N$46: IC1.20, R30.2
- new net N$47: IC1.6, R31.2
- new net N$49: R28.E, R30.1
- new net N$50: R19.1, R26.E
- new net N$52: C17.2, C23.1, C24.1, C50.2
- new net N$68: IC1.23, R50.1
- new net SW_MODE_A: SW1.3, SW1.4, U1.27
- new net SW_MODE_B: SW2.3, SW2.4, U1.29
- new net SW_MODE_C: SW3.3, SW3.4, U1.30
- net +3V3: now also C37.1, C39.1, C40.1, C42.1, L2.2, LED10.A, LED11.A, LED12.A, R26.B, R28.B, R29.B, U1.1, U1.17
- net +3V3_A: now also C10.1, C11.1, C30.1, C33.1, C9.1, IC3.16, U2.4, U3.8
- net ADC_TIME_SHAPE: now also U1.9
- net A_ADC: now also U1.10
- net A_CV: now also U1.6
- net A_GATE: now also U1.20
- net A_TRIG: now also U1.25
- net B_ADC: now also U1.11
- net B_CV: now also U1.7
- net B_GATE: now also U1.21
- net B_TRIG: now also U1.14
- net C_ADC: now also U1.12
- net C_CV: now also U1.8
- net C_GATE: now also U1.22
- net C_TRIG: now also U1.15
- net GND: now also C10.2, C11.2, C30.2, C33.2, C7.2, C8.2, C9.2, IC1.1, IC1.21, IC3.7, Q2.2, Q2.4, R50.2, U2.11, U3.4; no longer R26.E, R28.E, R29.E
- net N$1: now also R29.E, R31.1; no longer R19.1, R26.B
- net POTS_ADDR_A: now also U1.13
- net POTS_ADDR_B: now also U1.18
- net POTS_ADDR_C: now also U1.19
- net VCC: now also C17.1, C50.1, U4.4, U5.8; no longer IC3.16
- net VEE: now also C23.2, C24.2, U4.11, U5.4; no longer IC3.7
