File: moire.sch (EAGLE design)
At the start: 121 parts, among them IC2 LD2981ABU33, IC3 4051PW, IC5 LM4040B10, IC6 R-78E3.3-0.5, J1 PJ301_THONKICONN6, J10 PJ301_THONKICONN6, J11 PJ301_THONKICONN6, J12 PJ301_THONKICONN6, J2 PJ301_THONKICONN6, J3 PJ301_THONKICONN6, J4 PJ301_THONKICONN6, J5 PJ301_THONKICONN6, J6 PJ301_THONKICONN6, J7 PJ301_THONKICONN6, J8 PJ301_THONKICONN6, J9 PJ301_THONKICONN6, Q2 8MHz, U1 STM32F303K8T6, U2 MCP6004_SMD, U3 MCP6002_, U4 TL074_SMD, U5 TL072_SMD

Commit message: update sch
Parts:
- added C10, C17, C23, C24, C30, C33, C50, C8, C9: 100n, rcl:C-USC0402
- added C11, C7: 22u, rcl:C-USC1206
- added IC1: TLC59281DBQ, og-ics:TLC59281DBQ
- added L2: (no value), wuerth-elektronik:WE-CBF_0603
- added LED10, LED11, LED12: SSL-LX3059IGW-CA, og-leds:LED-BICOLOR-THROUGHHOLE-CA
- added R50: 10k, rcl:R-US_R0402
Connections:
- removed net A_LED_1: R19.2
- removed net B_LED_1: R30.2
- removed net C_LED_1: R31.2
- removed net GRN: LED7.GRN, LED8.GRN, LED9.GRN
- removed net N$102: R29LED.A, R31.1
- removed net N$103: R28LED.A, R30.1
- removed net RED: LED7.RED, LED8.RED, LED9.RED
- removed net SW_MODE_1: SW1.3, SW1.4
- removed net SW_MODE_2: SW2.3, SW2.4
- removed net SW_MODE_3: SW3.3, SW3.4
- new net LEDS_SCK: IC1.SCLK, U1.PB3
- new net LEDS_SIN: IC1.SIN, U1.PB5
- new net N$101: IC1.OUT4, LED7.GRN
- new net N$32: IC1.OUT6, LED8.GRN
- new net N$33: IC1.OUT5, LED7.RED
- new net N$34: IC1.OUT7, LED8.RED
- new net N$35: IC1.OUT2, LED9.RED
- new net N$36: IC1.OUT3, LED9.GRN
- new net N$37: IC1.OUT10, LED11.RED
- new net N$38: IC1.OUT11, LED11.GRN
- new net N$39: IC1.OUT8, LED10.GRN
- new net N$40: IC1.OUT12, LED12.RED
- new net N$42: IC1.OUT13, LED12.GRN
- new net N$43: IC1.OUT9, LED10.RED
- new net N$44: C7.1, C8.1, IC1.VCC, L2.1
- new net N$45: IC1.OUT14, R19.2
- new net N$46: IC1.OUT15, R30.2
- new net N$47: IC1.OUT1, R31.2
- new net N$49: R28LED.C, R30.1
- new net N$50: R19.1, R26LED.C
- new net N$52: C17.2, C23.1, C24.1, C50.2
- new net N$68: IC1.IREF, R50.1
- new net SW_MODE_A: SW1.3, SW1.4, U1.PB4
- new net SW_MODE_B: SW2.3, SW2.4, U1.PB6
- new net SW_MODE_C: SW3.3, SW3.4, U1.PB7
- net +3V3: now also L2.2, LED10.A, LED11.A, LED12.A, R26LED.A, R28LED.A, R29LED.A
- net +3V3_A: now also C10.1, C11.1, C30.1, C33.1, C9.1, IC3P.VCC, U2P.V+, U3P.V+
- net ADC_TIME_SHAPE: now also U1.PA3
- net A_ADC: now also U1.PA4
- net A_CV: now also U1.PA0
- net A_GATE: now also U1.PA10
- net A_TRIG: now also U1.PA15
- net B_ADC: now also U1.PA5
- net B_CV: now also U1.PA1
- net B_GATE: now also U1.PA11
- net B_TRIG: now also U1.PB0
- net C_ADC: now also U1.PA6
- net C_CV: now also U1.PA2
- net C_GATE: now also U1.PA12
- net C_TRIG: now also U1.PB1
- net GND: now also C10.2, C11.2, C30.2, C33.2, C7.2, C8.2, C9.2, IC1.BLANK, IC1.GND, IC3P.GND, IC3P.VEE, Q2G$2.LID1, Q2G$2.LID2, R50.2, U2P.V-, U3P.V-; no longer R26LED.C, R28LED.C, R29LED.C
- net N$1: now also R29LED.C, R31.1; no longer R19.1, R26LED.A
- net POTS_ADDR_A: now also U1.PA7
- net POTS_ADDR_B: now also U1.PA8
- net POTS_ADDR_C: now also U1.PA9
- net VCC: now also C17.1, C50.1, U4P.V+, U5P.V+
- net VEE: now also C23.2, C24.2, U4P.V-, U5P.V-
Other:
- moved on the sheet: C1, C2, C3, C34, C35, C36, C4, C5, C6, J10, J11, J12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
