File: moire_v1.1.brd (EAGLE design)
At the start: 39.4 x 106.7 mm, 137 parts, among them IC1 TLC59281DBQ, IC11 LM4040B25, IC2 ROF-78E3.3-0.5SMD, IC3 4051PW, IC4 LM324PW, IC7 LD2981ABU33, IC9 LM324PW, J1 PJ301_THONKICONN6, J10 PJ301_THONKICONN6, J11 PJ301_THONKICONN6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

Commit message: update brd
Parts:
- removed JP5: M05X2SMD, og-header:2X5-SMD
- added JP8: M05X2PTH, og-header:2X5-PTH
- moved IC9 1094.8 mm to (43.0, 68.6)
- moved L5 1036.0 mm to (48.7, 71.6)
- moved C30 1034.2 mm to (53.7, 79.0)
- moved C14 1033.4 mm to (42.8, 86.9)
- moved C31 1032.3 mm to (48.1, 79.3)
- moved C16 1029.6 mm to (49.9, 82.6)
- moved C21 1029.1 mm to (48.6, 86.4)
- moved L1 1028.0 mm to (49.0, 74.7)
- moved C18 1026.8 mm to (43.6, 82.0)
- moved C20 1025.6 mm to (61.1, 79.3)
- moved IC2 1017.5 mm to (60.3, 89.7)
- moved L4 1015.0 mm to (74.1, 56.9)
- moved D4 1006.3 mm to (43.8, 46.5)
- moved C15 1005.1 mm to (49.4, 46.7)
- moved L3 1004.1 mm to (49.1, 51.3)
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Connections:
- new net N$15: JP8.9
- new net N$17: JP8.1
- net GND: now also JP8.3, JP8.4, JP8.5, JP8.6, JP8.7, JP8.8; no longer JP5.3, JP5.4, JP5.5, JP5.6, JP5.7, JP5.8
- net N$18: now also JP8.10; no longer JP5.1, JP5.2
- net N$96: now also JP8.2; no longer JP5.10, JP5.9
