File: moire_v1.2.brd (EAGLE design)
At the start: 39.4 x 106.7 mm, 137 parts, among them IC1 TLC59281DBQ, IC11 LM4040B25, IC2 ROF-78E3.3-0.5SMD, IC3 4051PW, IC4 LM324PW, IC7 LD2981ABU33, IC9 LM324PW, J1 PJ301_THONKICONN6, J10 PJ301_THONKICONN6, J11 PJ301_THONKICONN6, J12 PJ301_THONKICONN6, J2 PJ301_THONKICONN6, J3 PJ301_THONKICONN6, J4 PJ301_THONKICONN6, J5 PJ301_THONKICONN6, J6 PJ301_THONKICONN6, J7 PJ301_THONKICONN6, J8 PJ301_THONKICONN6, J9 PJ301_THONKICONN6, Q2 8MHz, Q5 MMBT3904, Q6 MMBT3904, Q7 MMBT3904, U1 STM32F303K8T6, U2 MCP6004_SMD, U4 TL074_SMD

Commit message: update brd
Parts:
- removed C19, C30: 22u, rcl:C1206
- removed JP5: M05X2SMD, og-header:2X5-SMD
- added C5: 10u, rcl:PANASONIC_A
- added C6: 100n, rcl:C0402
- added JP8: M05X2PTH, og-header:2X5-PTH
- added R42: 10kB, og-pots:ALPS_POT_VERTICAL
- C15: value 100n -> 22u; device rcl:C0402 -> rcl:C1206
- IC2: value ROF-78E3.3-0.5SMD -> R-78E3.3-0.5; device og-vreg:ROF78EXX-0.5SMD -> og-vreg:WE78
- POT_A, POT_B, POT_C: device og-pots:ALPS_POT_VERTICAL_PS -> og-pots:ALPS_POT_VERTICAL
- R1, R10, R12, R13, R14, R16, R17, R20, R26, R28, R29, R4, R5, R51, R52, R53, R6, R66, R67, R68, R69, R70, R71, R8, R9: device rcl:R0402 -> rcl:R0603
- moved IC9 1099.3 mm to (73.3, 66.0), flipped to the bottom
- moved C15 1047.5 mm to (47.5, 90.4), flipped to the bottom
- moved C14 1037.7 mm to (73.5, 84.3), flipped to the bottom
- moved L5 1037.7 mm to (67.6, 69.1), flipped to the bottom
- moved L3 1037.6 mm to (57.7, 83.8), flipped to the bottom
- moved C31 1034.1 mm to (68.2, 76.7), flipped to the bottom
- moved C16 1030.7 mm to (66.4, 80.0), flipped to the bottom
- moved C18 1030.5 mm to (72.8, 79.5), flipped to the bottom
- moved C21 1030.4 mm to (67.7, 83.8), flipped to the bottom
- moved L1 1029.1 mm to (67.3, 72.1), flipped to the bottom
- moved C13 1024.1 mm to (52.6, 90.4), flipped to the bottom
- moved IC2 1023.5 mm to (49.0, 98.3), flipped to the bottom, turned to 270 degrees
- moved C20 1021.9 mm to (55.3, 76.7), flipped to the bottom
- moved D4 1010.3 mm to (72.5, 43.9), flipped to the bottom
- moved L4 1006.2 mm to (42.2, 54.4), flipped to the bottom
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Connections:
- removed net N$18: D3.A, JP5.1, JP5.2
- removed net N$96: D4.C, JP5.10, JP5.9
- removed net N$99: C19.1, IC2.1, L3.2
- new net +12V: D3.A, JP8.10
- new net -12V: D4.C, JP8.2
- new net N$15: JP8.9
- new net N$17: JP8.1
- new net N$66: C15.1, IC2.1, L3.2
- new net N$67: C13.1, L3.1
- net +3V3: now also C5.+, C6.1; no longer C15.1, C30.1
- net GND: now also C5.-, C6.2, JP8.3, JP8.4, JP8.5, JP8.6, JP8.7, JP8.8; no longer C19.2, C30.2, JP5.3, JP5.4, JP5.5, JP5.6, JP5.7, JP5.8
- net N$4: no longer C13.1, L3.1
