File: moire_v1.2_plc.brd (EAGLE design)
At the start: 39.4 x 106.7 mm, 137 parts, among them IC1 TLC59281DBQ, IC11 LM4040B25, IC2 ROF-78E3.3-0.5SMD, IC3 4051PW, IC4 LM324PW, IC7 LD2981ABU33, IC9 LM324PW, J1 PJ301_THONKICONN6, J10 PJ301_THONKICONN6, J11 PJ301_THONKICONN6, J12 PJ301_THONKICONN6, J2 PJ301_THONKICONN6, J3 PJ301_THONKICONN6, J4 PJ301_THONKICONN6, J5 PJ301_THONKICONN6, J6 PJ301_THONKICONN6, J7 PJ301_THONKICONN6, J8 PJ301_THONKICONN6, J9 PJ301_THONKICONN6, Q2 8MHz, Q5 MMBT3904, Q6 MMBT3904, Q7 MMBT3904, U1 STM32F303K8T6, U2 MCP6004_SMD, U4 TL074_SMD

Commit message: update brd
Parts:
- removed C19, C30: 22u, rcl:C1206
- removed IC4: LM324PW, og-linear:TSSOP14_065
- removed JP5: M05X2SMD, og-header:2X5-SMD
- added C5: 10u, rcl:PANASONIC_A
- added C6: 100n, rcl:C0402
- added JP8: M05X2PTH, og-header:2X5-PTH
- C15: value 100n -> 22u; device rcl:C0402 -> rcl:C1206
- IC2: value ROF-78E3.3-0.5SMD -> R-78E3.3-0.5; device og-vreg:ROF78EXX-0.5SMD -> og-vreg:WE78
- POT_A, POT_B, POT_C: device og-pots:ALPS_POT_VERTICAL_PS -> og-pots:ALPS_POT_VERTICAL
- R1, R10, R12, R13, R14, R16, R17, R20, R26, R28, R29, R4, R5, R51, R52, R53, R6, R66, R67, R68, R69, R70, R71, R8, R9: device rcl:R0402 -> rcl:R0603
- U$1: value ISL21010 -> VREF 1.5V
- moved C15 1058.1 mm to (36.1, 103.4), flipped to the bottom, turned to 270 degrees
- moved D4 1057.4 mm to (9.52, 105.2), flipped to the bottom, turned to 180 degrees
- moved L3 1053.7 mm to (32.5, 105.2), flipped to the bottom, turned to 180 degrees
- moved L1 1049.0 mm to (9.40, 102.6), flipped to the bottom, turned to 90 degrees
- moved L5 1048.1 mm to (7.37, 91.9), flipped to the bottom, turned to 90 degrees
- moved L4 1046.8 mm to (48.5, 94.5), flipped to the bottom, turned to 180 degrees
- moved C14 1044.8 mm to (16.8, 103.5), flipped to the bottom, turned to 270 degrees
- moved C18 1041.0 mm to (12.6, 102.1), flipped to the bottom
- moved C20 1039.8 mm to (59.1, 94.2), flipped to the bottom
- moved C21 1037.2 mm to (7.36, 101.5), flipped to the bottom, turned to 270 degrees
- moved C16 1034.8 mm to (7.36, 95.9), flipped to the bottom, turned to 270 degrees
- moved C31 1034.1 mm to (68.2, 76.7), flipped to the bottom
- moved D3 1034.0 mm to (3.18, 91.2), flipped to the bottom
- moved C13 1032.6 mm to (29.0, 103.4), flipped to the bottom, turned to 270 degrees
- moved IC9 1032.2 mm to (12.6, 11.2), flipped to the bottom
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Connections:
- removed net N$18: D3.A, JP5.1, JP5.2
- removed net N$96: D4.C, JP5.10, JP5.9
- removed net N$99: C19.1, IC2.1, L3.2
- removed net V+: IC9.4
- removed net V-: IC9.11
- new net +12V: D3.A, JP8.10, JP8.9
- new net -12V: D4.C, JP8.1, JP8.2
- new net N$66: C15.1, IC2.1, L3.2
- new net N$67: C13.1, L3.1
- net +3V3: now also C5.+, C6.1; no longer C15.1, C30.1
- net GND: now also C5.-, C6.2, IC9.11, JP8.3, JP8.4, JP8.5, JP8.6, JP8.7, JP8.8; no longer C19.2, C30.2, IC4.11, JP5.3, JP5.4, JP5.5, JP5.6, JP5.7, JP5.8
- net N$4: no longer C13.1, L3.1
- net VCC: now also IC9.4; no longer IC4.4

Commit message: update board
Parts:
- moved R1 74.5 mm to (12.8, 87.1)
- moved C31 60.0 mm to (8.26, 80.0)
- moved IC7 55.2 mm to (26.3, 73.4), turned to 180 degrees
- moved C34 45.8 mm to (5.33, 70.0), turned to 0 degrees
- moved C35 45.7 mm to (2.17, 58.7)
- moved C20 42.8 mm to (17.6, 104.9), turned to 180 degrees
- moved C10 42.7 mm to (25.5, 21.8), turned to 270 degrees
- moved R19 41.0 mm to (11.8, 44.2)
- moved C11 40.7 mm to (28.1, 21.8), turned to 270 degrees
- moved C9 40.5 mm to (23.0, 21.8), turned to 270 degrees
- moved C43 39.4 mm to (18.4, 51.8), turned to 270 degrees
- moved R21 39.3 mm to (6.74, 66.0)
- moved C8 38.8 mm to (29.3, 72.1)
- moved R22 37.3 mm to (6.35, 59.8), turned to 0 degrees
- moved L4 37.0 mm to (13.0, 104.9), turned to 0 degrees
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Routing:
- net N$5: track 0.00 -> 37.9 mm
- net VEE: track 0.00 -> 7.07 mm
- net VCC: track 0.00 -> 6.73 mm
- net -12V: track 0.00 -> 3.89 mm
- net N$4: track 0.00 -> 3.24 mm
- net +12V: track 0.00 -> 2.66 mm
- net N$3: track 0.00 -> 2.17 mm
