File: moire_v1.2_rtb.sch (EAGLE design)
At the start: 134 parts, among them IC1 TLC59281DBQ, IC11 LM4040B25, IC2 R-78E3.3-0.5, IC3 4051PW, IC7 LD2981ABU33, IC9 LM324PW, J1 PJ301_THONKICONN6, J10 PJ301_THONKICONN6, J11 PJ301_THONKICONN6, J12 PJ301_THONKICONN6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

Commit message: finish placement and begin routing
Parts:
- added JP2: (no value), DECADE-libraries20151104:M06SIP
Connections:
- removed net N$67: C13.1, L3.1
- net +3V3: now also JP2.4
- net +3V3_A: now also JP2.3
- net AREF_-2.5: now also JP2.2
- net GND: now also JP2.1
- net N$4: now also C13.1, L3.1
- net VCC: now also JP2.6
- net VEE: now also JP2.5
