File: moire_v1.3_rt.sch (EAGLE design)
At the start: 134 parts, among them IC1 TLC59281DBQ, IC11 LM4040B25, IC2 R-78E3.3-0.5, IC3 4051PW, IC7 LD2981ABU33, IC9 LM324PW, J1 PJ301_THONKICONN6, J10 PJ301_THONKICONN6, J11 PJ301_THONKICONN6, J12 PJ301_THONKICONN6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

Commit message: finish placement and begin routing
Connections:
- net N$17 renamed A_OUT
- net N$2 renamed C_GATE_OUT
- net N$20 renamed A_GATE_OUT
- net N$21 renamed A_CV_IN
- net N$22 renamed C_CV_IN
- net N$7 renamed B_OUT
- net N$86 renamed C_OUT
- removed net N$67: C13.1, L3.1
- net A_ADC: now also R33.2; no longer R47.2
- net A_CV: now also C28.2, R52.1, U2D.OUT; no longer C12.2, R5.1, U2A.OUT
- net A_GATE: now also R20.2; no longer R10.2
- net A_TRIG: now also Q7.C; no longer Q5.C
- net A_TRIG_IN: now also J6.3, R66.1; no longer J4.3, R67.1
- net C_ADC: now also R47.2; no longer R33.2
- net C_CV: now also C12.2, R5.1, U2A.OUT; no longer C28.2, R52.1, U2D.OUT
- net C_GATE: now also R10.2; no longer R20.2
- net C_TRIG: now also Q5.C; no longer Q7.C
- net C_TRIG_IN: now also J4.3, R67.1; no longer J6.3, R66.1
- net N$4: now also C13.1, L3.1
Other:
- moved on the sheet: C1, C12, C28, C3, D1, D2, IC9A, IC9C, J11, J12, J2, J4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
