File: moire_v1.4-wip.sch (EAGLE design)
At the start: 134 parts, among them IC1 TLC59281DBQ, IC11 LM4040B25, IC2 R-78E3.3-0.5, IC3 4051PW, IC7 LD2981ABU33, IC9 LM324PW, J1 PJ301_THONKICONN6, J10 PJ301_THONKICONN6, J11 PJ301_THONKICONN6, J12 PJ301_THONKICONN6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

Commit message: finish placement and begin routing
Parts:
- added U$1: 1X6-SMD-TESTPAD, CUSTOM:1X6-SMD-TESTPAD
Connections:
- removed net N$67: C13.1, L3.1
- net +3V3: now also U$1.P$3
- net +3V3_A: now also U$1.P$4
- net AREF_-2.5: now also U$1.P$5
- net GND: now also U$1.P$6
- net N$4: now also C13.1, L3.1
- net VCC: now also U$1.P$1
- net VEE: now also U$1.P$2
