File: moire_v1.4.brd (EAGLE design)
At the start: 39.4 x 106.7 mm, 134 parts, among them IC1 TLC59281DBQ, IC11 LM4040B25, IC2 R-78E3.3-0.5, IC3 4051PW, IC7 LD2981ABU33, IC9 LM324PW, J1 PJ301_THONKICONN6, J10 PJ301_THONKICONN6, J11 PJ301_THONKICONN6, J12 PJ301_THONKICONN6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

Commit message: finish placement and begin routing
Parts:
- added U$1: 1X6-SMD-TESTPAD, CUSTOM:6X1-SMD-TESTPAD
- moved R21 3.18 mm to (3.56, 56.6), turned to 0 degrees
- moved C35 1.70 mm to (2.79, 64.3)
- moved R4 1.52 mm to (35.3, 30.5)
- moved R31 1.27 mm to (35.8, 40.6)
- moved R70 1.27 mm to (29.7, 32.8)
- moved R67 1.05 mm to (35.3, 33.3)
- moved C11 1.02 mm to (2.54, 69.3)
- moved D2 1.02 mm to (32.3, 33.0)
- moved C20 0.92 mm to (16.5, 103.1)
- moved C23 0.80 mm to (7.37, 56.6)
- moved IC7 0.51 mm to (21.6, 103.1)
- moved Q2 0.36 mm to (6.35, 60.2)
Connections:
- removed net N$67: C13.1, L3.1
- net +3V3: now also U$1.3
- net +3V3_A: now also U$1.4
- net AREF_-2.5: now also U$1.5
- net GND: now also U$1.6
- net N$4: now also C13.1, L3.1
- net VCC: now also U$1.1
- net VEE: now also U$1.2
Routing:
- net +3V3: track 0.00 -> 106.9 mm, vias 0 -> 2
- net AREF_-2.5: track 0.00 -> 69.4 mm, vias 0 -> 2
- net N$4: track 0.00 -> 25.6 mm
- net VCC: track 0.00 -> 22.4 mm, vias 0 -> 1
- net VEE: track 0.00 -> 16.4 mm
- net +3V3_A: track 0.00 -> 8.11 mm
- net N$5: track 0.00 -> 5.95 mm
- net N$66: track 0.00 -> 5.92 mm
- net -12V: track 0.00 -> 3.94 mm
- net +12V: track 0.00 -> 2.78 mm
- net N$3: track 0.00 -> 2.07 mm
- added copper zone on layer 1, net GND
- added copper zone on layer 16, net GND
