File: moire_v1.5-routed.sch (EAGLE design)
At the start: 135 parts, among them IC1 R-78E3.3-0.5, IC100 LM324PW, IC101 TLC59281DBQ, IC102 4051PW, IC103 LM4040B25, IC104 LD2981ABU33, J1 PJ301_THONKICONN6, J10 PJ301_THONKICONN6, J11 PJ301_THONKICONN6, J12 PJ301_THONKICONN6, J2 PJ301_THONKICONN6, J3 PJ301_THONKICONN6, J4 PJ301_THONKICONN6, J5 PJ301_THONKICONN6, J6 PJ301_THONKICONN6, J7 PJ301_THONKICONN6, J8 PJ301_THONKICONN6, J9 PJ301_THONKICONN6, Q100 MMBT3904, Q101 MMBT3904, Q102 MMBT3904, Q103 8MHz, U100 MCP6004, U101 STM32F303K8T6, U102 TL074

Commit message: finishing touches
Parts:
- D1, D2: value 1N5819HW -> 1N5819
- IC2: value LD2981ABU33 -> LD2981
- renumbered C100 to C35, C101 to C34, C102 to C33, C103 to C32, C104 to C30, C105 to C29, C106 to C31, C107 to C24, C108 to C23, C109 to C28, C110 to C27, C111 to C26, C112 to C25, C113 to C14, C114 to C15, C115 to C20, C116 to C19, C117 to C18, C118 to C17, C119 to C22, C120 to C21, C121 to C16, C122 to C13, C123 to C11, C124 to C12, C125 to C8, C126 to C6, C127 to C7, C128 to C10, C129 to C9, C130 to C5, C131 to C1, C132 to C3, C133 to C2, C134 to C4, D100 to D5, D101 to D4, D102 to D3, D103 to D2, D104 to D1, IC100 to IC6, IC101 to IC5, IC102 to IC4, IC103 to IC3, IC104 to IC2, JP100 to JP2, JP101 to JP1, L100 to L5, L101 to L4, L102 to L1, L103 to L2, L104 to L3, Q100 to Q4, Q101 to Q3, Q102 to Q2, Q103 to Q1, R100 to R43, R101 to R42, R102 to R44, R103 to R47, R104 to R46, R105 to R41, R106 to R45, R107 to R40, R108 to R39, R109 to R38, R110 to R36, R111 to R35, R112 to R34, R113 to R37, R114 to R33, R115 to R26, R116 to R22, R117 to R21, R118 to R20, R119 to R32, R120 to R31, R121 to R25, R122 to R19, R123 to R30, R124 to R23, R125 to R29, R126 to R28, R127 to R18, R128 to R24, R129 to R27, R130 to R14, R131 to R15, R132 to R17, R133 to R13, R134 to R12, R135 to R11, R136 to R16, R137 to R8, R138 to R7, R139 to R10, R140 to R6, R141 to R9, R142 to R5, R143 to R4, R144 to R3, R145 to R2, R146 to R1, U100 to U2, U101 to U1, U102 to U3
Connections:
- net A_TRIG_IN: now also J3.3; no longer J5.3
- net B_CV_IN: now also J5.3; no longer J4.3
- net B_TRIG_IN: now also J2.3; no longer J3.3
- net N$21: now also J4.3; no longer J2.3
