File: moire_v1.7.brd (EAGLE design)
At the start: 39.4 x 106.7 mm, 135 parts, among them IC1 R-78E3.3-0.5, IC2 LD2981, IC3 LM4040B25, IC4 4051PW, IC5 TLC59281DBQ, IC6 LM324PW, J1 PJ301_THONKICONN6, J10 PJ301_THONKICONN6, J11 PJ301_THONKICONN6, J12 PJ301_THONKICONN6, J2 PJ301_THONKICONN6, J3 PJ301_THONKICONN6, J4 PJ301_THONKICONN6, J5 PJ301_THONKICONN6, J6 PJ301_THONKICONN6, J7 PJ301_THONKICONN6, J8 PJ301_THONKICONN6, J9 PJ301_THONKICONN6, Q1 8MHz, Q2 MMBT3904, Q3 MMBT3904, Q4 MMBT3904, U1 STM32F303K8T6, U2 MCP6004, U3 TL074

Commit message: finishing touches
Parts:
- C1, C10, C14, C16, C2, C3, C4, C5, C7, C9: device rcl:C1206 -> moire_v1.5-routed:RCL_C1206
- C11, C12, C13, C15, C17, C18, C19, C20, C21, C22, C23, C24, C25, C26, C27, C28, C29, C30, C31, C32, C33, C34, C35, C6: device rcl:C0603 -> moire_v1.5-routed:RCL_C0603
- C8: device rcl:PANASONIC_A -> moire_v1.5-routed:RCL_PANASONIC_A
- R1, R10, R11, R12, R13, R14, R15, R16, R17, R18, R19, R2, R20, R21, R22, R23, R24, R25, R26, R27, R28, R29, R3, R30, R31, R32, R33, R34, R35, R36, R37, R38, R39, R4, R40, R41, R42, R43, R44, R45, R46, R47, R5, R6, R7, R8, R9: device rcl:R0603 -> moire_v1.5-routed:RCL_R0603
- renumbered LED1 to A_OUT_LED, LED2 to B_OUT_LED, LED3 to C_OUT_LED
Other:
- board text added: "-2.5V"
- board text added: "1"
- board text added: "2"
- board text added: "3"
- board text added: "3V3"
- board text added: "3V3A"
- board text added: "4"
- board text added: "GND"
- board text added: "VCC"
- board text added: "VEE"
