File: moire_v2.1.brd (EAGLE design)
At the start: 39.4 x 100 mm, 141 parts, among them IC1 R-78E3.3-0.5, IC14 TL074PW, IC2 LD2981, IC3 LM4040B, IC4 4051PW, IC5 TLC59281DBQ, IC6 LM324PW, J1 PJ301_THONKICONN6, J10 PJ301_THONKICONN6, J11 PJ301_THONKICONN6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

Commit message: update board v2.1
Parts:
- IC14: value TL074PW -> LM324
- IC6: value LM324PW -> LM324
- R37, R38, R39, R40, R42, R43, R48, R49, R50: value 1.0k -> 1k

Commit message: update
Parts:
- IC14, IC6: value LM324 -> TL074PW
- IC2: value LD2981 -> AP7380; device og-vreg:SOT89 -> v-reg-custom:SOT89
- moved IC2 0.97 mm to (26.0, 78.7)
- moved R43 0.68 mm to (36.9, 7.59)
- moved C7 0.31 mm to (36.3, 80.4), turned to 0 degrees
- moved C6 0.18 mm to (37.0, 86.8)
- moved C8 0.10 mm to (30.9, 80.5)
Connections:
- net +3V3_A: now also IC2.3; no longer IC2.1
- net GND: now also IC2.1; no longer IC2.2
- net N$5: now also IC2.2, IC2.4; no longer IC2.3
Routing:
- net GND: track 104.7 -> 95.1 mm
- net N$59: track 118.0 -> 113.6 mm, vias 6 -> 4
- net N$58: track 110.3 -> 112.5 mm
- net +3V3_A: track 173.7 -> 175.1 mm
- net N$93: track 88.8 -> 89.9 mm
- net N$5: track 38.3 -> 37.6 mm, vias 5 -> 3
Other:
- board text added: "+"
