File: moire_v2.1.sch (EAGLE design)
At the start: 141 parts, among them IC1 R-78E3.3-0.5, IC14 TL074PW, IC2 LD2981, IC3 LM4040B, IC4 4051PW, IC5 TLC59281DBQ, IC6 LM324PW, J1 PJ301_THONKICONN6, J10 PJ301_THONKICONN6, J11 PJ301_THONKICONN6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

Commit message: update board v2.1
Parts:
- IC14: value TL074PW -> LM324
- IC6: value LM324PW -> LM324
- R37, R38, R39, R40, R42, R43, R48, R49, R50: value 1.0k -> 1k
Changed lines of the file:
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@@
 <part name="SW_C" library="SparkFun" deviceset="TAC_SWITCH" device="PTH"/>
 <part name="J10" library="og-pj301_variations" deviceset="PJ301_THONKICONN" device="6"/>
-<part name="R43" library="moire_v1.5-routed" deviceset="RCL_R-US_" device="R0603" value="1.0k"/>
+<part name="R43" library="moire_v1.5-routed" deviceset="RCL_R-US_" device="R0603" value="1k"/>
 <part name="R32" library="moire_v1.5-routed" deviceset="RCL_R-US_" device="R0603" value="100k"/>
 <part name="R31" library="moire_v1.5-routed" deviceset="RCL_R-US_" device="R0603" value="20k"/>
@@
 <part name="GND56" library="SparkFun" deviceset="GND" device=""/>
 <part name="GND30" library="SparkFun" deviceset="GND" device=""/>
-<part name="IC6" library="og-linear" deviceset="TL074" device="PW" value="LM324PW"/>
-<part name="R39" library="moire_v1.5-routed" deviceset="RCL_R-US_" device="R0603" value="1.0k"/>
+<part name="IC6" library="og-linear" deviceset="TL074" device="PW" value="LM324"/>
+<part name="R39" library="moire_v1.5-routed" deviceset="RCL_R-US_" device="R0603" value="1k"/>
 <part name="R44" library="moire_v1.5-routed" deviceset="RCL_R-US_" device="R0603" value="100k"/>
 <part name="R47" library="moire_v1.5-routed" deviceset="RCL_R-US_" device="R0603" value="69.8k"/>
 <part name="GND31" library="SparkFun" deviceset="GND" device=""/>
 <part name="R13" library="moire_v1.5-routed" deviceset="RCL_R-US_" device="R0603" value="10k"/>
-<part name="R38" library="moire_v1.5-routed" deviceset="RCL_R-US_" device="R0603" value="1.0k"/>
+<part name="R38" library="moire_v1.5-routed" deviceset="RCL_R-US_" device="R0603" value="1k"/>
 <part name="R41" library="moire_v1.5-routed" deviceset="RCL_R-US_" device="R0603" value="100k"/>
 <part name="R46" library="moire_v1.5-routed" deviceset="RCL_R-US_" device="R0603" value="69.8k"/>
 <part name="GND33" library="SparkFun" deviceset="GND" device=""/>
 <part name="R12" library="moire_v1.5-routed" deviceset="RCL_R-US_" device="R0603" value="10k"/>
-<part name="R37" library="moire_v1.5-routed" deviceset="RCL_R-US_" device="R0603" value="1.0k"/>
+<part name="R37" library="moire_v1.5-routed" deviceset="RCL_R-US_" device="R0603" value="1k"/>
 <part name="R36" library="moire_v1.5-routed" deviceset="RCL_R-US_" device="R0603" value="100k"/>
 <part name="R45" library="moire_v1.5-routed" deviceset="RCL_R-US_" device="R0603" value="69.8k"/>
@@
 <part name="R30" library="moire_v1.5-routed" deviceset="RCL_R-US_" device="R0603" value="30k"/>
 <part name="GND61" library="SparkFun" deviceset="GND" device=""/>
-<part name="R42" library="moire_v1.5-routed" deviceset="RCL_R-US_" device="R0603" value="1.0k"/>
+<part name="R42" library="moire_v1.5-routed" deviceset="RCL_R-US_" device="R0603" value="1k"/>
 <part name="R29" library="moire_v1.5-routed" deviceset="RCL_R-US_" device="R0603" value="100k"/>
 <part name="R28" library="moire_v1.5-routed" deviceset="RCL_R-US_" device="R0603" value="20k"/>
@@
 <part name="R27" library="moire_v1.5-routed" deviceset="RCL_R-US_" device="R0603" value="30k"/>
 <part name="GND62" library="SparkFun" deviceset="GND" device=""/>
-<part name="R40" library="moire_v1.5-routed" deviceset="RCL_R-US_" device="R0603" value="1.0k"/>
+<part name="R40" library="moire_v1.5-routed" deviceset="RCL_R-US_" device="R0603" value="1k"/>
 <part name="R35" library="moire_v1.5-routed" deviceset="RCL_R-US_" device="R0603" value="100k"/>
 <part name="R34" library="moire_v1.5-routed" deviceset="RCL_R-US_" device="R0603" value="20k"/>
@@
 <part name="LED2" library="og-leds" deviceset="LED-BICOLOR-SHARED-THROUGHHOLE" device="" value="WP937EGW"/>
 <part name="GND16" library="SparkFun" deviceset="GND" device=""/>
-<part name="IC14" library="linear" deviceset="TL074" device="PW"/>
+<part name="IC14" library="linear" deviceset="TL074" device="PW" value="LM324"/>
 <part name="GND39" library="SparkFun" deviceset="GND" device=""/>
 <part name="C36" library="moire_v1.5-routed" deviceset="RCL_C-US" device="C0603" value="100n"/>
 <part name="C37" library="moire_v1.5-routed" deviceset="RCL_C-US" device="C0603" value="100n"/>
-<part name="R48" library="moire_v1.5-routed" deviceset="RCL_R-US_" device="R0603" value="1.0k"/>
-<part name="R49" library="moire_v1.5-routed" deviceset="RCL_R-US_" device="R0603" value="1.0k"/>
-<part name="R50" library="moire_v1.5-routed" deviceset="RCL_R-US_" device="R0603" value="1.0k"/>
+<part name="R48" library="moire_v1.5-routed" deviceset="RCL_R-US_" device="R0603" value="1k"/>
+<part name="R49" library="moire_v1.5-routed" deviceset="RCL_R-US_" device="R0603" value="1k"/>
+<part name="R50" library="moire_v1.5-routed" deviceset="RCL_R-US_" device="R0603" value="1k"/>
 </parts>
 <sheets>

Commit message: update
Parts:
- IC14, IC6: value LM324 -> TL074PW
- IC2: value LD2981 -> AP7380; device og-vreg:LD2981ABU -> v-reg-custom:AP7380
Connections:
- net +3V3_A: now also IC2.OUT; no longer IC2.VO
- net N$5: now also IC2.IN; no longer IC2.VI
