File: moire_v2.2.sch (EAGLE design)
At the start: 142 parts, among them IC1 R-78E3.3-0.5, IC14 TL074PW, IC2 AP7380, IC3 LM4040B, IC4 4051PW, IC5 TLC59281DBQ, IC6 TL074PW, J1 PJ301_THONKICONN6, J10 PJ301_THONKICONN6, J11 PJ301_THONKICONN6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

Commit message: update 2.5
Connections:
- removed net SWDIO: JP2.2
- net C_CV: now also JP3.4
- net C_CV_SS: now also JP3.3
- net LEDS_SS: now also JP3.2
- net SWDIO_SS: now also JP2.2
Changed lines of the file:
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@@
 <wire x1="53.34" y1="-33.02" x2="55.88" y2="-33.02" width="0.1524" layer="91"/>
 <label x="53.34" y="-33.02" size="1.778" layer="95"/>
+<pinref part="JP3" gate="G$1" pin="4"/>
 </segment>
 </net>
@@
 </segment>
 </net>
-<net name="SWDIO" class="0">
-<segment>
-<wire x1="109.22" y1="-129.54" x2="111.76" y2="-129.54" width="0.1524" layer="91"/>
-<label x="111.76" y="-129.54" size="1.778" layer="95"/>
-<pinref part="JP2" gate="G$1" pin="2"/>
-</segment>
-</net>
 <net name="A_CV" class="0">
 <segment>
@@
 <wire x1="53.34" y1="-38.1" x2="55.88" y2="-38.1" width="0.1524" layer="91"/>
 <label x="53.34" y="-38.1" size="1.778" layer="95"/>
+<pinref part="JP3" gate="G$1" pin="2"/>
 </segment>
 </net>
@@
 <label x="53.34" y="-40.64" size="1.778" layer="95"/>
 </segment>
+<segment>
+<wire x1="109.22" y1="-129.54" x2="111.76" y2="-129.54" width="0.1524" layer="91"/>
+<label x="111.76" y="-129.54" size="1.778" layer="95"/>
+<pinref part="JP2" gate="G$1" pin="2"/>
+</segment>
 </net>
 <net name="C_CV_SS" class="0">
@@
 <wire x1="53.34" y1="-35.56" x2="55.88" y2="-35.56" width="0.1524" layer="91"/>
 <label x="53.34" y="-35.56" size="1.778" layer="95"/>
-</segment>
-</net>
+<pinref part="JP3" gate="G$1" pin="3"/>
+</segment>
+</net>
