File: moire_v2.4.sch (EAGLE design)
At the start: 142 parts, among them IC1 R-78E3.3-0.5, IC14 TL074PW, IC2 AP7380, IC3 LM4040B, IC4 4051PW, IC5 TLC59281DBQ, IC6 TL074PW, J1 PJ301_THONKICONN6, J10 PJ301_THONKICONN6, J11 PJ301_THONKICONN6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

Commit message: update 2.5
Parts:
- renumbered LED1 to LED_OUT_2, LED2 to LED_OUT_3, LED3 to LED_OUT_1
Connections:
- removed net SWDIO: JP2.2
- net C_CV: now also JP3.4
- net C_CV_SS: now also JP3.3
- net LEDS_SS: now also JP3.2
- net N$19: no longer IC14C.-IN
- net N$52: no longer IC14C.+IN
- net N$60: no longer IC14C.OUT
- net N$84: no longer IC14A.+IN
- net N$85: no longer IC14A.OUT
- net N$93: no longer IC14A.-IN
- net SWDIO_SS: now also JP2.2
Other:
- moved on the sheet: IC14A, IC14C
