File: moire_v2.5.sch (EAGLE design)
At the start: 142 parts, among them IC1 R-78E3.3-0.5, IC14 TL074PW, IC2 AP7380, IC3 LM4040B, IC4 4051PW, IC5 TLC59281DBQ, IC6 TL074PW, J1 PJ301_THONKICONN6, J10 PJ301_THONKICONN6, J11 PJ301_THONKICONN6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

Commit message: update 2.5
Parts:
- D3, D4, D5: device moire_v1.7:DIODE_DIODE-SOD523 -> moire_v1.7:DIODE_DIODE-SOD323-R
- R27, R33: value 30k -> 40k
- R29, R35: value 100k -> 140k
- renumbered LED1 to LED_OUT_2, LED2 to LED_OUT_3, LED3 to LED_OUT_1
Connections:
- net A_ADC renamed C_DAC
- net B_ADC renamed B_DAC
- net C_ADC renamed A_DAC
- net N$13 renamed B_GATE_OUT
- net N$2 renamed A_GATE_OUT
- net N$20 renamed C_GATE_OUT
- removed net N$27 (its old number): SLD_ALED.A, SLD_BLED.A, SLD_CLED.A
- removed net SWDIO: JP2.2
- net +3V3: now also SLD_ALED.A, SLD_BLED.A, SLD_CLED.A
- net C_CV: now also JP3.4
- net C_CV_SS: now also JP3.3
- net LEDS_SS: now also JP3.2
- net N$19: no longer IC14C.-IN
- net N$52: no longer IC14C.+IN
- net N$60: no longer IC14C.OUT
- net N$84: no longer IC14A.+IN
- net N$85: no longer IC14A.OUT
- net N$93: no longer IC14A.-IN
- net SWDIO_SS: now also JP2.2
Other:
- moved on the sheet: IC14A, IC14C, R15, R16, R17, SLD_ALED, SLD_BLED, SLD_CLED
