File: moire_v2.6.brd (EAGLE design)
At the start: 39.4 x 100 mm, 145 parts, among them IC1 R-78E3.3-0.5, IC14 TL074PW, IC2 AP7380, IC3 LM4040B, IC4 4051PW, IC5 TLC59281DBQ, IC6 TL074PW, J1 PJ301_THONKICONN6, J10 PJ301_THONKICONN6, J11 PJ301_THONKICONN6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

Commit message: update 2.7
Parts:
- added LDAC: 0, moire_v1.5-routed:RCL_R0603
- moved U3 0.53 mm to (6.12, 50.8)
- moved MCU_DAC 0.18 mm to (12.7, 52.2)
Connections:
- removed net B_DAC: R28.2, U1.11, U4.3
- removed net N$2: J9.P2
- removed net N$47: U4.6
- new net B_DAC_LDAC: LDAC.2, R28.2, U1.11, U4.13, U4.3
- net +3V3: now also LDAC.1; no longer U4.13
- net A_LED: now also IC14.8
- net C_LED: now also IC14.1
- net N$19: now also IC14.10
- net N$52: now also IC14.9
- net N$84: now also IC14.2
- net N$93: now also IC14.3
Routing:
- net SPI_SCK: track 144.8 -> 34.4 mm
- net B_DAC_LDAC: track 0.00 -> 90.8 mm, vias 0 -> 10
- net B_DAC: track 74.3 -> 0.00 mm, vias 7 -> 0
- net C_DAC_SS: track 69.5 -> 20.3 mm, vias 4 -> 2
- net N$52: track 12.8 -> 43.0 mm, vias 1 -> 3
- net A_LED: track 0.00 -> 28.3 mm, vias 0 -> 5
- net N$19: track 65.4 -> 83.5 mm, vias 6 -> 8
- net N$93: track 79.8 -> 92.1 mm, vias 3 -> 5
- net N$84: track 3.35 -> 11.0 mm, vias 0 -> 1
- net N$29: track 56.8 -> 61.4 mm
- net B_CV: track 19.2 -> 23.2 mm
- net C_LED: track 0.00 -> 3.50 mm
- net +3V3: track 240.9 -> 242.9 mm
- net N$64: track 43.1 -> 44.2 mm
- net VCC: track 196.6 -> 195.9 mm
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