File: moire_v2.7.sch (EAGLE design)
At the start: 146 parts, among them IC1 R-78E3.3-0.5, IC14 TL074PW, IC2 AP7380, IC3 LM4040B, IC4 4051PW, IC5 TLC59281DBQ, IC6 TL074PW, J1 PJ301_THONKICONN6, J10 PJ301_THONKICONN6, J11 PJ301_THONKICONN6, J12 PJ301_THONKICONN6, J2 PJ301_THONKICONN6, J3 PJ301_THONKICONN6, J4 PJ301_THONKICONN6, J5 PJ301_THONKICONN6, J6 PJ301_THONKICONN6, J7 PJ301_THONKICONN6, J8 PJ301_THONKICONN6, J9 PJ301_THONKICONN6, Q1 8MHz, Q2 MMBT3904, Q3 MMBT3904, Q4 MMBT3904, U1 STM32F303K8T6, U2 MCP6004, U3 TL074, U4 MAX5715

Commit message: update 2.7
Parts:
- removed IC14: TL074PW, linear:TL074PW
- removed IC6: TL074PW, og-linear:TL074PW
- removed JP3: (no value), SparkFun:M04PTH
- removed LDAC, MCU_DAC: 0, moire_v1.5-routed:RCL_R-US_R0603
- removed U4: MAX5715, MAX5715BAUD:MAX5715BAUD
- added C39: 100n, rcl:C-USC0603
- added C40: 22u, rcl:CPOL-USC
- added C41: 470n, rcl:C-USC0603
- added D9: BAT54S, diode:DIODE_2CACA-SOT23
- added IC7: DAC8164, og-dac:DAC8564
- added IC8: TL074, linear:TL074PW
- added IC9: LM324, og-linear:TL074PW
- added R51, R52, R53: 10k, moire_v1.5-routed:RCL_R-US_R0603
- C38: device moire_v1.5-routed:RCL_C-USC0603 -> rcl:C-USC0603
- R27, R33: value 40k -> 30k
- R29, R35: value 140k -> 100k
- U3: value TL074 -> TL072; device MusicThingModular:TL074_SMD -> MusicThingModular:TL072TSSOP
Connections:
- net N$32 renamed RED_C
- net N$33 renamed GRN_C
- net N$34 renamed RED_B
- net N$35 renamed GRN_B
- net N$36 renamed RED_A
- net N$37 renamed GRN_A
- removed net A_CV_SS: JP3.3, U1.PA2
- removed net A_DAC: R34.2, U1.PA6, U4.OUTA
- removed net B_DAC_LDAC: LDAC.2, R28.2, U1.PA5, U4.OUTB, U4.VDDIO
- removed net C_DAC: MCU_DAC.1, R31.2, U4.OUTC
- removed net C_DAC_SS: MCU_DAC.2, U1.PA4, U4.CSB
- removed net N$31: IC14D.+IN, IC14D.OUT
- removed net SWDIO_SS: JP2.2, JP3.1, U1.PA13
- new net DAC_A: IC7.OUTA, R34.2
- new net DAC_B: IC7.OUTB, R28.2
- new net DAC_C: IC7.OUTC, R31.2
- new net DAC_SS: IC7.SYNC, U1.PA6
- new net N$13: J1.2, R51.2
- new net N$17: J3.2, R53.2
- new net NORMALIZATION_PROBE: D9.AC, R51.1, R52.1, R53.1, U1.PA4
- new net SWDIO: JP2.2, U1.PA13
- new net VREF: C41.1, IC7.VREFH
- net +3V3: now also C39.1, D9.C, IC7.DVDD; no longer LDAC.1, U4.*LDAC
- net +3V3_A: now also C40.+, IC7.AVDD; no longer U4.VDD
- net A_CV: now also U1.PA2; no longer IC4A.X6, JP3.4
- net A_LED: now also IC8D.OUT; no longer IC14C.OUT
- net B_LED: now also U3A.OUT; no longer IC14B.OUT
- net C_LED: now also U3B.OUT; no longer IC14A.OUT
- net GND: now also C39.2, C40.-, C41.2, D9.A, IC7.A0, IC7.A1, IC7.ENABLE, IC7.GND, IC7.LDAC, IC7.VREFL, IC8A.-IN, IC8B.-IN, IC8C.+IN, IC9D.-IN, IC9P.V-; no longer IC14D.-IN, IC6D.+IN, IC6P.V-, J1.2, J2.2, J3.2, U3A.+IN, U3B.+IN, U3C.+IN, U3D.+IN, U4.GND
- net LEDS_SS: now also U1.PA5; no longer JP3.2
- net N$14: now also J2.2, R52.2; no longer U3D.-IN, U3D.OUT
- net N$15: now also IC8B.OUT, U3A.-IN; no longer IC14B.+IN, U3B.OUT
- net N$16: now also IC9A.OUT; no longer IC6A.OUT
- net N$18: now also IC8C.-IN; no longer U3C.-IN
- net N$19: now also IC8C.OUT, IC8D.-IN; no longer IC14C.+IN, U3C.OUT
- net N$24: now also IC9A.+IN; no longer IC6A.+IN
- net N$25: now also IC9A.-IN; no longer IC6A.-IN
- net N$26: now also IC9B.OUT; no longer IC6B.OUT
- net N$28: now also IC9B.+IN; no longer IC6B.+IN
- net N$29: now also IC9B.-IN; no longer IC6B.-IN
- net N$30: now also IC9C.OUT; no longer IC6C.OUT
- net N$40: now also U3A.+IN; no longer IC14B.-IN
- net N$52: now also IC8D.+IN; no longer IC14C.-IN
- net N$6: now also IC9D.+IN, IC9D.OUT; no longer IC6D.-IN, IC6D.OUT
- net N$61: now also IC9C.-IN; no longer IC6C.+IN
- net N$64: now also IC9C.+IN; no longer IC6C.-IN
- net N$8: now also IC8B.+IN; no longer U3B.-IN
- net N$84: now also U3B.+IN; no longer IC14A.-IN
- net N$87: now also IC8A.+IN; no longer U3A.-IN
- net N$93: now also IC8A.OUT, U3B.-IN; no longer IC14A.+IN, U3A.OUT
- net SPI_MOSI: now also IC7.IN; no longer U4.DIN
- net SPI_SCK: now also IC7.SCK; no longer U4.SCLK
- net VCC: now also IC8P.V+, IC9P.V+; no longer IC14P.V+, IC6P.V+
- net VEE: now also IC8P.V-; no longer IC14P.V-
Other:
- moved on the sheet: C28, C29, D3, D4, D5, J1, J2, J3, Q2, Q3, Q4, R18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
